File: pcb/detector-opamp.sch (EAGLE design)
At the start: 14 parts, among them IC1 OPA2725D

Commit message: circuit as built
Parts:
- removed C2: 2p2, adafruit:C-USC0603K
- removed R6: 220k, adafruit:R-US_R0402
- R3: value 680k -> 100k
Connections:
- net N$2: no longer C2.2
- net N$3: no longer C2.1
- net N$6: no longer R6.1
- net N$7: no longer R6.2
Changed lines of the file:
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@@
 <?xml version="1.0" encoding="utf-8"?>
 <!DOCTYPE eagle SYSTEM "eagle.dtd">
-<eagle version="6.3">
+<eagle version="7.6.0">
 <drawing>
 <settings>
@@
 <part name="D1" library="opto-trans-siemens" deviceset="BPW32" device="" value="BPW34"/>
 <part name="C1" library="adafruit" deviceset="C-US" device="C0603K" value="100n"/>
-<part name="C2" library="adafruit" deviceset="C-US" device="C0603K" value="2p2"/>
 <part name="C3" library="adafruit" deviceset="C-US" device="C0603K" value="100n"/>
 <part name="R1" library="adafruit" deviceset="R-US_" device="R0402" value="18k"/>
 <part name="R2" library="adafruit" deviceset="R-US_" device="R0402" value="27k"/>
-<part name="R3" library="adafruit" deviceset="R-US_" device="R0402" value="680k"/>
+<part name="R3" library="adafruit" deviceset="R-US_" device="R0402" value="100k"/>
 <part name="R4" library="adafruit" deviceset="R-US_" device="R0402" value="10k"/>
 <part name="R5" library="adafruit" deviceset="R-US_" device="R0402" value="1k"/>
-<part name="R6" library="adafruit" deviceset="R-US_" device="R0402" value="220k"/>
 <part name="R8" library="adafruit" deviceset="R-US_" device="R0402" value="47"/>
 <part name="C4" library="adafruit" deviceset="C-US" device="C0603K" value="100n"/>
@@
 </instance>
 <instance part="C1" gate="G$1" x="50.8" y="149.86"/>
-<instance part="C2" gate="G$1" x="83.82" y="132.08" rot="R90"/>
 <instance part="C3" gate="G$1" x="99.06" y="160.02" rot="R90"/>
 <instance part="R1" gate="G$1" x="43.18" y="175.26" rot="R90"/>
@@
 <instance part="R4" gate="G$1" x="106.68" y="180.34" rot="R90"/>
 <instance part="R5" gate="G$1" x="114.3" y="180.34" rot="R90"/>
-<instance part="R6" gate="G$1" x="124.46" y="175.26"/>
 <instance part="R8" gate="G$1" x="142.24" y="162.56" rot="R180"/>
 <instance part="C4" gate="G$1" x="88.9" y="172.72" rot="R90"/>
@@
 <pinref part="C3" gate="G$1" pin="1"/>
 <wire x1="91.44" y1="160.02" x2="93.98" y2="160.02" width="0.1524" layer="91"/>
-<pinref part="C2" gate="G$1" pin="2"/>
 <wire x1="93.98" y1="160.02" x2="96.52" y2="160.02" width="0.1524" layer="91"/>
 <wire x1="88.9" y1="132.08" x2="93.98" y2="132.08" width="0.1524" layer="91"/>
@@
 <wire x1="78.74" y1="142.24" x2="73.66" y2="142.24" width="0.1524" layer="91"/>
 <wire x1="73.66" y1="142.24" x2="73.66" y2="157.48" width="0.1524" layer="91"/>
-<pinref part="C2" gate="G$1" pin="1"/>
 <wire x1="81.28" y1="132.08" x2="73.66" y2="132.08" width="0.1524" layer="91"/>
 <wire x1="73.66" y1="132.08" x2="73.66" y2="142.24" width="0.1524" layer="91"/>
@@
 <wire x1="116.84" y1="165.1" x2="114.3" y2="165.1" width="0.1524" layer="91"/>
 <wire x1="114.3" y1="165.1" x2="114.3" y2="175.26" width="0.1524" layer="91"/>
-<pinref part="R6" gate="G$1" pin="1"/>
 <wire x1="114.3" y1="175.26" x2="119.38" y2="175.26" width="0.1524" layer="91"/>
 <pinref part="R5" gate="G$1" pin="1"/>
@@
 <net name="N$7" class="0">
 <segment>
-<pinref part="R6" gate="G$1" pin="2"/>
 <wire x1="129.54" y1="175.26" x2="134.62" y2="175.26" width="0.1524" layer="91"/>
 <wire x1="134.62" y1="175.26" x2="134.62" y2="162.56" width="0.1524" layer="91"/>
