File: pcb/detector-discrete.sch (EAGLE design)
At the start: 49 parts, among them Q1 2N3906, Q2 2N3906, Q3 2N3906, T1 2N3904, T2 2N3904, T3 2N3904

Commit message: reorg slightly for clarity
Parts:
- added TP2: PTR1B1,27, testpad:PTR1B1,27
Connections:
- net N$18: now also TP2.TP
Other:
- moved on the sheet: C11, C12, C13, C5, IC1, Q3, R18, R19, R20, R21, R22, R23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

Commit message: more formatting tweaks
Other:
- note added: "Comparator seems to be optional? Output at TP2 seems good enough for input into Teensy input capture."
- moved on the sheet: C1, R20, R21, TP2
Changed lines of the file:
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@@
 <sheet>
 <plain>
+<text x="137.16" y="-25.4" size="1.778" layer="91">Comparator seems to be optional?
+Output at TP2 seems good enough for
+input into Teensy input capture.</text>
 </plain>
 <instances>
@@
 <attribute name="VALUE" x="40.64" y="68.58" size="1.778" layer="96"/>
 </instance>
-<instance part="T2" gate="G1" x="119.38" y="63.5"/>
+<instance part="T2" gate="G1" x="119.38" y="63.5" smashed="yes">
+<attribute name="NAME" x="124.46" y="63.5" size="1.778" layer="95"/>
+<attribute name="VALUE" x="124.46" y="60.96" size="1.778" layer="96"/>
+</instance>
 <instance part="Q1" gate="G$1" x="50.8" y="81.28" smashed="yes">
-<attribute name="NAME" x="45.72" y="83.82" size="1.778" layer="95"/>
-<attribute name="VALUE" x="43.18" y="76.2" size="1.778" layer="96"/>
+<attribute name="NAME" x="55.88" y="81.28" size="1.778" layer="95"/>
+<attribute name="VALUE" x="55.88" y="78.74" size="1.778" layer="96"/>
 </instance>
-<instance part="C1" gate="G$1" x="-2.54" y="99.06" rot="R90"/>
+<instance part="C1" gate="G$1" x="0" y="99.06" rot="R90"/>
 <instance part="C2" gate="G$1" x="63.5" y="91.44" rot="R180"/>
 <instance part="C3" gate="G$1" x="30.48" y="40.64" rot="R270"/>
@@
 <instance part="R18" gate="G$1" x="43.18" y="22.86" rot="R270"/>
 <instance part="R19" gate="G$1" x="43.18" y="7.62" rot="R270"/>
-<instance part="R20" gate="G$1" x="12.7" y="5.08" rot="R270"/>
-<instance part="R21" gate="G$1" x="12.7" y="-17.78" rot="R270"/>
+<instance part="R20" gate="G$1" x="12.7" y="7.62" rot="R270"/>
+<instance part="R21" gate="G$1" x="12.7" y="-15.24" rot="R270"/>
 <instance part="R22" gate="G$1" x="35.56" y="0"/>
 <instance part="R23" gate="G$1" x="58.42" y="-15.24" rot="R270"/>
@@
 <instance part="IC1" gate="G$1" x="127" y="-10.16"/>
 <instance part="+3V2" gate="G$1" x="43.18" y="33.02"/>
-<instance part="GND12" gate="1" x="12.7" y="-25.4"/>
+<instance part="GND12" gate="1" x="12.7" y="-22.86"/>
 <instance part="GND13" gate="1" x="27.94" y="-12.7"/>
 <instance part="GND14" gate="1" x="43.18" y="-22.86"/>
@@
 <instance part="+3V3" gate="G$1" x="104.14" y="-15.24"/>
 <instance part="+3V4" gate="G$1" x="127" y="7.62"/>
-<instance part="TP2" gate="G$1" x="83.82" y="-10.16"/>
+<instance part="TP2" gate="G$1" x="81.28" y="-10.16"/>
 </instances>
 <busses>
@@
 <pinref part="C1" gate="G$1" pin="2"/>
 <wire x1="10.16" y1="96.52" x2="10.16" y2="99.06" width="0.1524" layer="91"/>
-<wire x1="10.16" y1="99.06" x2="2.54" y2="99.06" width="0.1524" layer="91"/>
+<wire x1="10.16" y1="99.06" x2="5.08" y2="99.06" width="0.1524" layer="91"/>
 <pinref part="R3" gate="G$1" pin="2"/>
 <wire x1="12.7" y1="99.06" x2="10.16" y2="99.06" width="0.1524" layer="91"/>
@@
 <pinref part="C1" gate="G$1" pin="1"/>
 <pinref part="GND3" gate="1" pin="GND"/>
+<wire x1="-2.54" y1="99.06" x2="-5.08" y2="99.06" width="0.1524" layer="91"/>
 </segment>
 <segment>
@@
 <pinref part="R21" gate="G$1" pin="1"/>
 <wire x1="12.7" y1="-5.08" x2="-5.08" y2="-5.08" width="0.1524" layer="91"/>
-<wire x1="12.7" y1="0" x2="12.7" y2="-5.08" width="0.1524" layer="91"/>
+<wire x1="12.7" y1="2.54" x2="12.7" y2="-5.08" width="0.1524" layer="91"/>
 <junction x="12.7" y="-5.08"/>
-<wire x1="12.7" y1="-5.08" x2="12.7" y2="-12.7" width="0.1524" layer="91"/>
+<wire x1="12.7" y1="-5.08" x2="12.7" y2="-10.16" width="0.1524" layer="91"/>
 </segment>
 </net>
@@
 <pinref part="R20" gate="G$1" pin="1"/>
 <wire x1="43.18" y1="15.24" x2="12.7" y2="15.24" width="0.1524" layer="91"/>
-<wire x1="12.7" y1="15.24" x2="12.7" y2="10.16" width="0.1524" layer="91"/>
+<wire x1="12.7" y1="15.24" x2="12.7" y2="12.7" width="0.1524" layer="91"/>
 <pinref part="C11" gate="G$1" pin="1"/>
 <wire x1="43.18" y1="15.24" x2="58.42" y2="15.24" width="0.1524" layer="91"/>
@@
 <wire x1="58.42" y1="-5.08" x2="58.42" y2="-7.62" width="0.1524" layer="91"/>
 <wire x1="58.42" y1="-7.62" x2="58.42" y2="-10.16" width="0.1524" layer="91"/>
-<wire x1="58.42" y1="-7.62" x2="83.82" y2="-7.62" width="0.1524" layer="91"/>
+<wire x1="58.42" y1="-7.62" x2="81.28" y2="-7.62" width="0.1524" layer="91"/>
 <pinref part="R29" gate="G$1" pin="1"/>
 <junction x="58.42" y="-7.62"/>
 <pinref part="TP2" gate="G$1" pin="TP"/>
-<wire x1="83.82" y1="-7.62" x2="99.06" y2="-7.62" width="0.1524" layer="91"/>
-<junction x="83.82" y="-7.62"/>
+<wire x1="81.28" y1="-7.62" x2="99.06" y2="-7.62" width="0.1524" layer="91"/>
+<junction x="81.28" y="-7.62"/>
 </segment>
 </net>
@@
 </schematic>
 </drawing>
+<compatibility>
+<note version="6.3" minversion="6.2.2" severity="warning">
+Since Version 6.2.2 text objects can contain more than one line,
+which will not be processed correctly with this version.
+</note>
+</compatibility>
 </eagle>
